File: PCBs/RFM69HCW_v7.kicad_pcb (KiCad board)
At the start: 4 copper layers, 65.1 x 30.1 mm, 12 parts

Commit message: Add code
Parts:
- moved G*** 29.5 mm to (163.7, 94.9)
Other:
- board text added: "TwinRF69"
